File: source/template/template.kicad_pcb (KiCad board)
At the start: 2 copper layers, 0 parts

Commit message: update to kicad 8.99 2024-04-02
Parts:
- added REF**: KiCad-Logo_40mm_SilkScreen, Symbol:KiCad-Logo_40mm_SilkScreen, F.Cu at (160.0, 53.0)
- added REF**: KiCad-Logo_40mm_Copper, Symbol:KiCad-Logo_40mm_Copper, B.Cu at (160.0, 53.0)
Other:
- board outline added: 120 x 70 mm
- board text added: "Template"
